File: kicad/headphone-silencer.kicad_sch (KiCad schematic)
At the start: 6 parts, among them J1 AudioJack3, J2 AudioJack3

Commit message: Add pdfs
Parts:
- J1, J2: value AudioJack3 -> Kycon STX-3150-3C-1
Other:
- note added: "Input impedance Z_IN ≈ 10 Ω Output impedance Z_OUT ≈ 1 Ω J1, J2 = 3.5 mm audio jack"
- company: (none) -> Thomas Birbacher
- title: (none) -> HS1 Headphone Silencer
- moved on the sheet: J1, J2, R1, R2, R3, R4
